File: project/_driver.kicad_sch (KiCad schematic)
At the start: 23 parts, among them U201 74HC595, U202 ULN2803A, U203 74HC595, U204 ULN2803A

Commit message: routing somewhat done
Parts:
- added C203, C205: 10u/50v, Capacitor_SMD:C_0805_2012Metric_Pad1.18x1.45mm_HandSolder, symbol Device:C
- renumbered C203 to C204
Connections:
- net 24V: now also C203.1, C205.1
- net GND: now also C203.2, C205.2
Changed lines of the file:
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@@
     (company "makerspace.lt")
   )
+  (junction (at 157.48 88.9) (diameter 0) (color 0 0 0 0)
+  )
+  (junction (at 157.48 132.08) (diameter 0) (color 0 0 0 0)
+  )
   (wire (pts (xy 154.94 114.3) (xy 168.91 114.3))
     (stroke (width 0) (type default) (color 0 0 0 0))
@@
     (stroke (width 0) (type default) (color 0 0 0 0))
   )
+  (wire (pts (xy 157.48 88.9) (xy 181.61 88.9))
+    (stroke (width 0) (type default) (color 0 0 0 0))
+  )
   (wire (pts (xy 134.62 114.3) (xy 124.46 114.3))
     (stroke (width 0) (type default) (color 0 0 0 0))
@@
     (stroke (width 0) (type default) (color 0 0 0 0))
   )
-  (wire (pts (xy 154.94 132.08) (xy 181.61 132.08))
+  (wire (pts (xy 154.94 132.08) (xy 157.48 132.08))
     (stroke (width 0) (type default) (color 0 0 0 0))
   )
@@
     (stroke (width 0) (type default) (color 0 0 0 0))
   )
+  (wire (pts (xy 157.48 132.08) (xy 181.61 132.08))
+    (stroke (width 0) (type default) (color 0 0 0 0))
+  )
   (wire (pts (xy 134.62 121.92) (xy 124.46 121.92))
     (stroke (width 0) (type default) (color 0 0 0 0))
@@
     (stroke (width 0) (type default) (color 0 0 0 0))
   )
-  (wire (pts (xy 154.94 88.9) (xy 181.61 88.9))
+  (wire (pts (xy 154.94 88.9) (xy 157.48 88.9))
     (stroke (width 0) (type default) (color 0 0 0 0))
   )
@@
     (effects (font (size 1.27 1.27)) (justify left))
   )
+  (hierarchical_label "GND" (shape bidirectional) (at 157.48 139.7 270)
+    (effects (font (size 1.27 1.27)) (justify right))
+  )
   (hierarchical_label "R4" (shape output) (at 181.61 78.74 0)
     (effects (font (size 1.27 1.27)) (justify left))
@@
   (hierarchical_label "R13" (shape output) (at 181.61 124.46 0)
     (effects (font (size 1.27 1.27)) (justify left))
+  )
+  (hierarchical_label "GND" (shape bidirectional) (at 157.48 96.52 270)
+    (effects (font (size 1.27 1.27)) (justify right))
   )
   (hierarchical_label "5V" (shape input) (at 104.14 119.38 180)
@@
     (pin "2")
   )
+  (symbol (lib_id "Device:C") (at 157.48 135.89 0) (unit 1)
+    (in_bom yes) (on_board yes)
+    (property "Reference" "C205" (id 0) (at 158.75 133.35 0)
+      (effects (font (size 1.27 1.27)) (justify left))
+    )
+    (property "Value" "10u/50v" (id 1) (at 158.75 138.43 0)
+      (effects (font (size 1.27 1.27)) (justify left))
+    )
+    (property "Footprint" "Capacitor_SMD:C_0805_2012Metric_Pad1.18x1.45mm_HandSolder" (id 2) (at 158.4452 139.7 0)
+      (effects (font (size 1.27 1.27)) hide)
+    )
+    (property "Datasheet" "https://www.lcsc.com/datasheet/lcsc_datasheet_2411041759_Murata-Electronics-GRM21BR61H106KE43L_C440198.pdf" (id 3) (at 157.48 135.89 0)
+      (effects (font (size 1.27 1.27)) hide)
+    )
+    (property "jlc-part-type" "B" (id 4) (at 157.48 135.89 0)
+      (effects (font (size 1.27 1.27)) hide)
+    )
+    (property "lcsc#" "C440198" (id 5) (at 157.48 135.89 0)
+      (effects (font (size 1.27 1.27)) hide)
+    )
+    (pin "1")
+    (pin "2")
+  )
   (symbol (lib_id "Device:C") (at 125.73 105.41 90) (unit 1)
     (in_bom yes) (on_board yes)
-    (property "Reference" "C203" (id 0) (at 132.08 102.87 90)
+    (property "Reference" "C204" (id 0) (at 132.08 102.87 90)
       (effects (font (size 1.27 1.27)) (justify left))
     )
@@
       (effects (font (size 1.27 1.27)) hide)
     )
+    (pin "1")
+    (pin "2")
+  )
+  (symbol (lib_id "Device:C") (at 157.48 92.71 0) (unit 1)
+    (in_bom yes) (on_board yes)
+    (property "Reference" "C203" (id 0) (at 158.75 90.17 0)
+      (effects (font (size 1.27 1.27)) (justify left))
+    )
+    (property "Value" "10u/50v" (id 1) (at 158.75 95.25 0)
+      (effects (font (size 1.27 1.27)) (justify left))
+    )
+    (property "Footprint" "Capacitor_SMD:C_0805_2012Metric_Pad1.18x1.45mm_HandSolder" (id 2) (at 158.4452 96.52 0)
+      (effects (font (size 1.27 1.27)) hide)
+    )
+    (property "Datasheet" "https://www.lcsc.com/datasheet/lcsc_datasheet_2411041759_Murata-Electronics-GRM21BR61H106KE43L_C440198.pdf" (id 3) (at 157.48 92.71 0)
+      (effects (font (size 1.27 1.27)) hide)
+    )
+    (property "jlc-part-type" "B" (id 4) (at 157.48 92.71 0)
+      (effects (font (size 1.27 1.27)) hide)
+    )
+    (property "lcsc#" "C440198" (id 5) (at 157.48 92.71 0)
+      (effects (font (size 1.27 1.27)) hide)
+    )

Commit message: fixing silk and bom and generating prod/doc files
Parts:
- D201, D202, D203, D204, D205, D206, D207, D208, D209, D210, D211, D212, D213, D214, D215, D216: jlc-part-type (none) -> E; lcsc# (none) -> C5356080
- U202, U204: jlc-part-type (none) -> E; lcsc# (none) -> C845537
Connections:
- net O_DATA: now reaches U201.9 (QH'), U203.14 (SER)
- no-connect marks 0 -> 1
Changed lines of the file:
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@@
   (junction (at 157.48 132.08) (diameter 0) (color 0 0 0 0)
   )
+  (junction (at 93.98 52.07) (diameter 0) (color 0 0 0 0)
+  )
+  (no_connect (at 124.46 134.62))
   (wire (pts (xy 154.94 114.3) (xy 168.91 114.3))
     (stroke (width 0) (type default) (color 0 0 0 0))
@@
   (wire (pts (xy 118.11 97.79) (xy 118.11 102.87))
     (stroke (width 0) (type default) (color 0 0 0 0))
+  )
+  (label "O_DATA" (at 110.49 102.87 180)
+    (effects (font (size 1.27 1.27)) (justify right bottom))
   )
   (hierarchical_label "R8" (shape output) (at 181.61 111.76 0)
@@
       (effects (font (size 1.27 1.27)) hide)
     )
+    (property "jlc-part-type" "E" (id 4) (at 161.29 83.82 0)
+      (effects (font (size 1.27 1.27)) hide)
+    )
+    (property "lcsc#" "C5356080" (id 5) (at 161.29 83.82 0)
+      (effects (font (size 1.27 1.27)) hide)
+    )
     (pin "1")
     (pin "2")
@@
       (effects (font (size 1.27 1.27)) hide)
     )
+    (property "jlc-part-type" "E" (id 4) (at 172.72 114.3 0)
+      (effects (font (size 1.27 1.27)) hide)
+    )
+    (property "lcsc#" "C5356080" (id 5) (at 172.72 114.3 0)
+      (effects (font (size 1.27 1.27)) hide)
+    )
     (pin "1")
     (pin "2")
@@
       (effects (font (size 1.27 1.27)) hide)
     )
-    (property "Datasheet" "~" (id 3) (at 125.73 105.41 0)
+    (property "Datasheet" "https://www.lcsc.com/datasheet/lcsc_datasheet_2304140030_Samsung-Electro-Mechanics-CL21B104KCFNNNE_C28233.pdf" (id 3) (at 125.73 105.41 0)
       (effects (font (size 1.27 1.27)) hide)
     )
@@
       (effects (font (size 1.27 1.27)) hide)
     )
+    (property "jlc-part-type" "E" (id 4) (at 161.29 68.58 0)
+      (effects (font (size 1.27 1.27)) hide)
+    )
+    (property "lcsc#" "C5356080" (id 5) (at 161.29 68.58 0)
+      (effects (font (size 1.27 1.27)) hide)
+    )
     (pin "1")
     (pin "2")
@@
       (effects (font (size 1.27 1.27)) hide)
     )
-    (pin "1")
-    (pin "2")
+    (property "jlc-part-type" "E" (id 4) (at 161.29 116.84 0)
+      (effects (font (size 1.27 1.27)) hide)
+    )
+    (property "lcsc#" "C5356080" (id 5) (at 161.29 116.84 0)
+      (effects (font (size 1.27 1.27)) hide)
+    )
+    (pin "1")
+    (pin "2")
+  )
+  (symbol (lib_id "power:PWR_FLAG") (at 93.98 52.07 0) (unit 1)
+    (in_bom yes) (on_board yes) (fields_autoplaced)
+    (property "Reference" "#FLG0201" (id 0) (at 93.98 50.165 0)
+      (effects (font (size 1.27 1.27)) hide)
+    )
+    (property "Value" "PWR_FLAG" (id 1) (at 93.98 46.99 0))
+    (property "Footprint" "" (id 2) (at 93.98 52.07 0)
+      (effects (font (size 1.27 1.27)) hide)
+    )
+    (property "Datasheet" "~" (id 3) (at 93.98 52.07 0)
+      (effects (font (size 1.27 1.27)) hide)
+    )
+    (pin "1")
   )
   (symbol (lib_id "Device:LED") (at 172.72 124.46 0) (mirror x) (unit 1)
@@
       (effects (font (size 1.27 1.27)) hide)
     )
+    (property "jlc-part-type" "E" (id 4) (at 172.72 124.46 0)
+      (effects (font (size 1.27 1.27)) hide)
+    )
+    (property "lcsc#" "C5356080" (id 5) (at 172.72 124.46 0)
+      (effects (font (size 1.27 1.27)) hide)
+    )
     (pin "1")
     (pin "2")
@@
       (effects (font (size 1.27 1.27)) hide)
     )
+    (property "jlc-part-type" "E" (id 4) (at 161.29 121.92 0)
+      (effects (font (size 1.27 1.27)) hide)
+    )
+    (property "lcsc#" "C5356080" (id 5) (at 161.29 121.92 0)
+      (effects (font (size 1.27 1.27)) hide)
+    )
     (pin "1")
     (pin "2")
@@
       (effects (font (size 1.27 1.27)) hide)
     )
+    (property "jlc-part-type" "E" (id 4) (at 161.29 111.76 0)
+      (effects (font (size 1.27 1.27)) hide)
+    )
+    (property "lcsc#" "C5356080" (id 5) (at 161.29 111.76 0)
+      (effects (font (size 1.27 1.27)) hide)
+    )
     (pin "1")
     (pin "2")
@@
       (effects (font (size 1.27 1.27)) hide)
     )
+    (property "jlc-part-type" "E" (id 4) (at 172.72 81.28 0)
+      (effects (font (size 1.27 1.27)) hide)
+    )
+    (property "lcsc#" "C5356080" (id 5) (at 172.72 81.28 0)
+      (effects (font (size 1.27 1.27)) hide)
+    )
     (pin "1")
     (pin "2")
@@
       (effects (font (size 1.27 1.27)) hide)
     )
+    (property "jlc-part-type" "E" (id 4) (at 172.72 76.2 0)
+      (effects (font (size 1.27 1.27)) hide)
+    )
+    (property "lcsc#" "C5356080" (id 5) (at 172.72 76.2 0)
+      (effects (font (size 1.27 1.27)) hide)
+    )
     (pin "1")
     (pin "2")
@@
     )
     (property "Datasheet" "https://www.lcsc.com/datasheet/lcsc_datasheet_2302091130_TOGIALED-TJ-S3216SWETNPLC2R-A5_C5356080.pdf" (id 3) (at 172.72 86.36 0)
+      (effects (font (size 1.27 1.27)) hide)
+    )
+    (property "jlc-part-type" "E" (id 4) (at 172.72 86.36 0)
+      (effects (font (size 1.27 1.27)) hide)
+    )
+    (property "lcsc#" "C5356080" (id 5) (at 172.72 86.36 0)
       (effects (font (size 1.27 1.27)) hide)
     )
@@
       (effects (font (size 1.27 1.27)) hide)
     )
+    (property "jlc-part-type" "E" (id 4) (at 172.72 129.54 0)
+      (effects (font (size 1.27 1.27)) hide)
+    )
+    (property "lcsc#" "C5356080" (id 5) (at 172.72 129.54 0)
+      (effects (font (size 1.27 1.27)) hide)
+    )
     (pin "1")
     (pin "2")
@@
       (effects (font (size 1.27 1.27)) hide)
     )
+    (property "jlc-part-type" "E" (id 4) (at 172.72 119.38 0)
+      (effects (font (size 1.27 1.27)) hide)
+    )
+    (property "lcsc#" "C5356080" (id 5) (at 172.72 119.38 0)
+      (effects (font (size 1.27 1.27)) hide)
+    )
     (pin "1")
     (pin "2")
@@
       (effects (font (size 1.27 1.27)) hide)
     )
+    (property "jlc-part-type" "E" (id 4) (at 161.29 78.74 0)
+      (effects (font (size 1.27 1.27)) hide)
+    )
+    (property "lcsc#" "C5356080" (id 5) (at 161.29 78.74 0)
+      (effects (font (size 1.27 1.27)) hide)
+    )
     (pin "1")
     (pin "2")
@@
       (effects (font (size 1.27 1.27)) hide)
     )
+    (property "jlc-part-type" "E" (id 4) (at 161.29 73.66 0)
+      (effects (font (size 1.27 1.27)) hide)
+    )
+    (property "lcsc#" "C5356080" (id 5) (at 161.29 73.66 0)
+      (effects (font (size 1.27 1.27)) hide)
+    )
     (pin "1")
     (pin "2")
@@
       (effects (font (size 1.27 1.27)) hide)
     )
+    (property "jlc-part-type" "E" (id 4) (at 172.72 71.12 0)
+      (effects (font (size 1.27 1.27)) hide)
+    )
+    (property "lcsc#" "C5356080" (id 5) (at 172.72 71.12 0)
+      (effects (font (size 1.27 1.27)) hide)
+    )
     (pin "1")
     (pin "2")
@@
       (effects (font (size 1.27 1.27)) hide)
     )
+    (property "jlc-part-type" "E" (id 4) (at 161.29 127 0)
+      (effects (font (size 1.27 1.27)) hide)
+    )
+    (property "lcsc#" "C5356080" (id 5) (at 161.29 127 0)
+      (effects (font (size 1.27 1.27)) hide)
+    )
     (pin "1")
     (pin "2")
@@
       (effects (font (size 1.27 1.27)) hide)
     )
-    (property "Datasheet" "~" (id 3) (at 125.73 60.96 0)
+    (property "Datasheet" "https://www.lcsc.com/datasheet/lcsc_datasheet_2304140030_Samsung-Electro-Mechanics-CL21B104KCFNNNE_C28233.pdf" (id 3) (at 125.73 60.96 0)
       (effects (font (size 1.27 1.27)) hide)
     )
@@
     )
     (property "Datasheet" "https://www.lcsc.com/datasheet/lcsc_datasheet_2311091738_UMW-Youtai-Semiconductor-Co---Ltd--ULN2803A_C845537.pdf" (id 3) (at 147.32 76.2 0)
+      (effects (font (size 1.27 1.27)) hide)
+    )
+    (property "jlc-part-type" "E" (id 4) (at 144.78 81.28 0)
+      (effects (font (size 1.27 1.27)) hide)
+    )
+    (property "lcsc#" "C845537" (id 5) (at 144.78 81.28 0)
       (effects (font (size 1.27 1.27)) hide)
     )
@@
       (effects (font (size 1.27 1.27)) hide)
     )
+    (property "jlc-part-type" "E" (id 4) (at 144.78 124.46 0)
+      (effects (font (size 1.27 1.27)) hide)
+    )
+    (property "lcsc#" "C845537" (id 5) (at 144.78 124.46 0)
+      (effects (font (size 1.27 1.27)) hide)
+    )
