File: project/project.kicad_sch (KiCad schematic)
At the start: 26 parts, among them J101 OUT, J102 IN, J103 FFC, J104 Back, J105 Front, Q101 DTC143Z, SW101 SW_DIP_x04, U101 GX101, U102 GX101

Commit message: routing somewhat done
Parts:
- H101, H102: footprint MountingHole:MountingHole_3.2mm_M3_Pad_Via -> -local:MountingHole_3.2mm_M3_Pad_Via
Connections:
- net F_GND is gone; now on net B_GND: C101.2, D101.1 (K), D102.1 (K), D103.1 (K), J103.16 (Pin_16), J103.18 (Pin_18), J103.20 (Pin_20), J103.22 (Pin_22), SW101.5, SW101.6, SW101.7, SW101.8, U101.2 (GND), U101.5 (ADD0)
- net GND is gone; now on net B_GND: J103.MP (MountPin)
- net B_24V: now also J104.16 (Pin_16)
- net B_3V3: now also J104.2 (Pin_2)
- net B_5V: now also J104.14 (Pin_14)
- net B_CAN_LED: now also J104.15 (Pin_15)
- net B_CLOCK: now also J104.12 (Pin_12)
- net B_DATA: now also J104.8 (Pin_8)
- net B_GND: now also H101.1, H102.1, H103.1, H104.1, J104.10 (Pin_10), J104.4 (Pin_4), J104.6 (Pin_6), J105.10 (Pin_10), J105.4 (Pin_4), J105.6 (Pin_6)
- net B_LATCH: now also J104.13 (Pin_13)
- net B_SCL: now also J104.3 (Pin_3)
- net B_SDA: now also J104.1 (Pin_1)
- net F_24V: now also J105.16 (Pin_16)
- net F_3V3: now also J105.2 (Pin_2)
- net F_5V: now also J105.14 (Pin_14)
- net F_CAN_LED: now also J105.15 (Pin_15)
- net F_CLOCK: now also J105.12 (Pin_12)
- net F_DATA: now also J105.8 (Pin_8)
- net F_LATCH: now also J105.13 (Pin_13)
- net F_SCL: now also J105.3 (Pin_3)
- net F_SDA: now also J105.1 (Pin_1)
Other:
- moved on the sheet: H101, H102, H103, H104

Commit message: fixing silk and bom and generating prod/doc files
Parts:
- removed Q101: DTC143Z, Package_TO_SOT_SMD:SOT-23, symbol Transistor_BJT:DTC143Z
- D101: value 24V -> RED; jlc-part-type (none) -> E; lcsc# (none) -> C5356080
- D102: value 5V -> RED; jlc-part-type (none) -> E; lcsc# (none) -> C5356080
- D103: value 3V3 -> RED; jlc-part-type (none) -> E; lcsc# (none) -> C5356080
- D104: value CAN -> RED; jlc-part-type (none) -> E; lcsc# (none) -> C5356080
- H101, H102: jlc-part-type (none) -> -
- H103, H104: jlc-part-type (none) -> X; lcsc# (none) -> C30182781
- J101: value OUT -> BUS; jlc-part-type (none) -> E; lcsc# (none) -> C880556
- J102: value IN -> BUS; jlc-part-type (none) -> E; lcsc# (none) -> C880556
- J104: jlc-part-type (none) -> E; lcsc# (none) -> C3975153
- J105: jlc-part-type (none) -> E; lcsc# (none) -> C5160782
- R101: lcsc# (none) -> C17713
- R102: lcsc# (none) -> C17414
- R103, R104, R105: lcsc# (none) -> C17673
- SW101: jlc-part-type (none) -> E; lcsc# (none) -> C976366
- U101, U102: jlc-part-type (none) -> E; lcsc# (none) -> C5441728
Connections:
- net B_GND: no longer C101.2, D101.1 (K), D102.1 (K), D103.1 (K), H103.1, H104.1, J103.16 (Pin_16), J103.18 (Pin_18), J103.20 (Pin_20), J103.22 (Pin_22), J103.MP (MountPin), J105.10 (Pin_10), J105.4 (Pin_4), J105.6 (Pin_6), SW101.5, SW101.6, SW101.7, SW101.8, U101.2 (GND), U101.5 (ADD0)
- new net F_GND: C101.2, D101.1 (K), D102.1 (K), D103.1 (K), H103.1, H104.1, J103.16 (Pin_16), J103.18 (Pin_18), J103.20 (Pin_20), J103.22 (Pin_22), J103.MP (MountPin), J105.10 (Pin_10), J105.4 (Pin_4), J105.6 (Pin_6), SW101.5, SW101.6, SW101.7, SW101.8, U101.2 (GND), U101.5 (ADD0)
Other:
- note added: "BACK"
- note added: "FRONT"
- moved on the sheet: J102

Commit message: bom fixes
Parts:
- added BOM101, BOM102: 1x4 screw plug, symbol Mechanical:Heatsink
Changed lines of the file:
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@@
   (title_block
     (title "WormControl-Relay15x5t15-ControlUI")
-    (date "2024-12-16")
+    (date "2024-12-19")
     (rev "0.1")
     (company "makerspace.lt")
@@
     (pin "1")
     (pin "2")
+  )
+  (symbol (lib_id "Mechanical:Heatsink") (at 26.67 121.92 90) (unit 1)
+    (in_bom yes) (on_board no)
+    (property "Reference" "BOM102" (id 0) (at 25.4 115.57 0)
+      (effects (font (size 1.27 1.27)) (justify left) hide)
+    )
+    (property "Value" "1x4 screw plug" (id 1) (at 43.18 121.92 90)
+      (effects (font (size 1.27 1.27)) (justify left))
+    )
+    (property "Footprint" "" (id 2) (at 26.67 121.6152 0)
+      (effects (font (size 1.27 1.27)) hide)
+    )
+    (property "Datasheet" "https://www.lcsc.com/datasheet/lcsc_datasheet_2304140030_Ningbo-Xinlaiya-Elec--XY2500F-F-3-5-4P_C560232.pdf" (id 3) (at 26.67 121.6152 0)
+      (effects (font (size 1.27 1.27)) hide)
+    )
+    (property "jlc-part-type" "E" (id 4) (at 26.67 121.92 0)
+      (effects (font (size 1.27 1.27)) hide)
+    )
+    (property "lcsc#" "C560232" (id 5) (at 26.67 121.92 0)
+      (effects (font (size 1.27 1.27)) hide)
+    )
   )
   (symbol (lib_id "Connector_Generic:Conn_01x16") (at 140.97 107.95 0) (mirror y) (unit 1)
@@
     (pin "1")
   )
+  (symbol (lib_id "Mechanical:Heatsink") (at 26.67 114.3 90) (unit 1)
+    (in_bom yes) (on_board no)
+    (property "Reference" "BOM101" (id 0) (at 25.4 107.95 0)
+      (effects (font (size 1.27 1.27)) (justify left) hide)
+    )
+    (property "Value" "1x4 screw plug" (id 1) (at 43.18 114.3 90)
+      (effects (font (size 1.27 1.27)) (justify left))
+    )
+    (property "Footprint" "" (id 2) (at 26.67 113.9952 0)
+      (effects (font (size 1.27 1.27)) hide)
+    )
+    (property "Datasheet" "https://www.lcsc.com/datasheet/lcsc_datasheet_2304140030_Ningbo-Xinlaiya-Elec--XY2500F-F-3-5-4P_C560232.pdf" (id 3) (at 26.67 113.9952 0)
+      (effects (font (size 1.27 1.27)) hide)
+    )
+    (property "jlc-part-type" "E" (id 4) (at 26.67 114.3 0)
+      (effects (font (size 1.27 1.27)) hide)
+    )
+    (property "lcsc#" "C560232" (id 5) (at 26.67 114.3 0)
+      (effects (font (size 1.27 1.27)) hide)
+    )
+  )
   (symbol (lib_id "Device:C") (at 95.25 158.75 0) (unit 1)
     (in_bom yes) (on_board yes)
@@
       (reference "#FLG0302") (unit 1) (value "PWR_FLAG") (footprint "")
     )
+    (path "/e080c4e6-20eb-4f29-bc7d-396f34edf8a9"
+      (reference "BOM101") (unit 1) (value "1x4 screw plug") (footprint "")
+    )
+    (path "/23dc5562-667b-4eea-8075-97f2d71954cb"
+      (reference "BOM102") (unit 1) (value "1x4 screw plug") (footprint "")
+    )
     (path "/af92851c-b649-444d-afad-7ba4c5709184"

Commit message: adding some 3d models
Parts:
- J101, J102: footprint Connector_Phoenix_MC:PhoenixContact_MCV_1,5_4-G-3.5_1x04_P3.50mm_Vertical -> -local:PhoenixContact_MCV_1,5_4-G-3.5_1x04_P3.50mm_Vertical
Changed lines of the file:
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@@
       (effects (font (size 1.27 1.27)) (justify left))
     )
-    (property "Footprint" "Connector_Phoenix_MC:PhoenixContact_MCV_1,5_4-G-3.5_1x04_P3.50mm_Vertical" (id 2) (at 38.1 74.93 0)
+    (property "Footprint" "-local:PhoenixContact_MCV_1,5_4-G-3.5_1x04_P3.50mm_Vertical" (id 2) (at 38.1 74.93 0)
       (effects (font (size 1.27 1.27)) hide)
     )
@@
     (property "Reference" "J101" (id 0) (at 20.32 66.04 0))
     (property "Value" "BUS" (id 1) (at 20.32 68.58 0))
-    (property "Footprint" "Connector_Phoenix_MC:PhoenixContact_MCV_1,5_4-G-3.5_1x04_P3.50mm_Vertical" (id 2) (at 20.32 74.93 0)
+    (property "Footprint" "-local:PhoenixContact_MCV_1,5_4-G-3.5_1x04_P3.50mm_Vertical" (id 2) (at 20.32 74.93 0)
       (effects (font (size 1.27 1.27)) hide)
     )
@@
     )
     (path "/da7504b3-69f1-4142-8ce9-4deec2331551"
-      (reference "J101") (unit 1) (value "BUS") (footprint "Connector_Phoenix_MC:PhoenixContact_MCV_1,5_4-G-3.5_1x04_P3.50mm_Vertical")
+      (reference "J101") (unit 1) (value "BUS") (footprint "-local:PhoenixContact_MCV_1,5_4-G-3.5_1x04_P3.50mm_Vertical")
     )
     (path "/b4491cbc-9a3c-4eaa-b841-783c4b62d70b"
-      (reference "J102") (unit 1) (value "BUS") (footprint "Connector_Phoenix_MC:PhoenixContact_MCV_1,5_4-G-3.5_1x04_P3.50mm_Vertical")
+      (reference "J102") (unit 1) (value "BUS") (footprint "-local:PhoenixContact_MCV_1,5_4-G-3.5_1x04_P3.50mm_Vertical")
     )
     (path "/3ccb35ae-5136-4707-82f3-14ec5132a1c1"

Commit message: replacing connector and fixing models
Parts:
- BOM101, BOM102: lcsc# C560232 -> C7603442
Changed lines of the file:
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@@
       (effects (font (size 1.27 1.27)) hide)
     )
-    (property "Datasheet" "https://www.lcsc.com/datasheet/lcsc_datasheet_2304140030_Ningbo-Xinlaiya-Elec--XY2500F-F-3-5-4P_C560232.pdf" (id 3) (at 26.67 121.6152 0)
+    (property "Datasheet" "https://www.lcsc.com/datasheet/lcsc_datasheet_2309070925_DEGSON-15EDGKN-3-5-04P-14-00A-H_C7603442.pdf" (id 3) (at 26.67 121.6152 0)
       (effects (font (size 1.27 1.27)) hide)
     )
@@
       (effects (font (size 1.27 1.27)) hide)
     )
-    (property "lcsc#" "C560232" (id 5) (at 26.67 121.92 0)
+    (property "lcsc#" "C7603442" (id 5) (at 26.67 121.92 0)
       (effects (font (size 1.27 1.27)) hide)
     )
@@
       (effects (font (size 1.27 1.27)) hide)
     )
-    (property "Datasheet" "https://www.lcsc.com/datasheet/lcsc_datasheet_2304140030_Ningbo-Xinlaiya-Elec--XY2500F-F-3-5-4P_C560232.pdf" (id 3) (at 26.67 113.9952 0)
+    (property "Datasheet" "https://www.lcsc.com/datasheet/lcsc_datasheet_2309070925_DEGSON-15EDGKN-3-5-04P-14-00A-H_C7603442.pdf" (id 3) (at 26.67 113.9952 0)
       (effects (font (size 1.27 1.27)) hide)
     )
@@
       (effects (font (size 1.27 1.27)) hide)
     )
-    (property "lcsc#" "C560232" (id 5) (at 26.67 114.3 0)
-      (effects (font (size 1.27 1.27)) hide)
-    )
+    (property "lcsc#" "C7603442" (id 5) (at 26.67 114.3 0)
+      (effects (font (size 1.27 1.27)) hide)
+    )

Commit message: few fixes and bumping up version
* reordering id bits
* moving silkscreen around
* adding hole in the center tab
Connections:
- net B_ID1: now also J104.11 (Pin_11); no longer J104.5 (Pin_5)
- net B_ID2: now also J104.9 (Pin_9); no longer J104.7 (Pin_7)
- net B_ID3: now also J104.7 (Pin_7); no longer J104.9 (Pin_9)
- net B_ID4: now also J104.5 (Pin_5); no longer J104.11 (Pin_11)
- net F_ID1: now also J105.11 (Pin_11), SW101.1; no longer J105.5 (Pin_5), SW101.4
- net F_ID2: now also J105.9 (Pin_9), SW101.2; no longer J105.7 (Pin_7), SW101.3
- net F_ID3: now also J105.7 (Pin_7), SW101.3; no longer J105.9 (Pin_9), SW101.2
- net F_ID4: now also J105.5 (Pin_5), SW101.4; no longer J105.11 (Pin_11), SW101.1

Commit message: improvements for next prototype
* buck makes 6v now
* using LDO for 5v with over voltage disable
* using LDO for 3v3
* adding zener to 24v led to stop it from glowing from 5v USB
* added 0.2mm heigt for USB port hole
* both buttons now 15mm height
Parts:
- added D101: 6V8, Diode_SMD:D_SOD-323_HandSoldering, symbol Device:D_Zener
- renumbered C102 to C101, C101 to C102, D101 to D102, D102 to D103, D103 to D104, D104 to D105, J104 to J103, J105 to J104, J103 to J105, U102 to U101, U101 to U102
Connections:
- net F_24V: now also D101.1 (K); no longer R101.2
- new net: D101.2 (A), R101.2
